File: analog_front_end_v2.kicad_sch (KiCad schematic)
At the start: 201 parts, among them J1 Conn_Coaxial, J3 Conn_01x01_Socket, J4 Conn_01x01_Socket, T1 JTX-4-10T_, U1 ADL5531, U10 PMOD 2x6, U11 LP2985-5.0, U12 LP2985-5.0, U13 ADA4899-1YRDZ, U14 MAX 735, U15 LP2985-2.5, U16 LT5546, U18 PAT1220-C-0DB, U19 PAT1220-C-0DB, U2 ADL5531, U20 PAT1220-C-0DB, U21 PAT1220-C-0DB, U22 LP2985-3.3, U23 PMOD 2x6, U24 ADA4899-1YRDZ, U3 ADL5531, U4 ADA4899-1YRDZ, U5 ADF4360-9, U6 LT5546, U7 LT5546, U8 ADA4899-1YRDZ, U9 PMOD 2x6

Commit message: Improve regulation in power supplies and hookup 7 segment supply in sch, last part remaining is where to connect the 7segs to the Arty S7
Parts:
- added C94: 10u_50V, Capacitor_SMD:C_1206_3216Metric, symbol Device:C
- added C95: 47u_16V, Capacitor_SMD:C_1206_3216Metric, symbol Device:C
- added U17, U25, U26, U27: KCSA02-123, Display_7Segment:KCSC02-123, symbol Display_Character:KCSA02-123
- added U28: LM1117MP-3.3, Package_TO_SOT_SMD:SOT-223-3_TabPin2, symbol Regulator_Linear:LM1117MP-3.3
Connections:
- net 3.3V: no longer C24.2, C25.1, C26.1, R1.2, R2.2
- net GND: now also C94.1, C95.1, U28.1 (GND)
- net VIN: now also C94.2, U28.3 (VI)
- new net 3.3V_IQ_DEMOD: C24.2, C25.1, C26.1, R1.2, R2.2
- new net 3V3_SEVEN_SEG: C95.2, U17.3 (CA), U17.8 (CA), U25.3 (CA), U25.8 (CA), U26.3 (CA), U26.8 (CA), U27.3 (CA), U27.8 (CA), U28.2 (VO)
- new net SEVEN_SEG_1_A: U17.7 (A)
- new net SEVEN_SEG_1_B: U17.6 (B)
- new net SEVEN_SEG_1_C: U17.4 (C)
- new net SEVEN_SEG_1_D: U17.2 (D)
- new net SEVEN_SEG_1_DP: U17.5 (DP)
- new net SEVEN_SEG_1_E: U17.1 (E)
- new net SEVEN_SEG_1_F: U17.9 (F)
- new net SEVEN_SEG_1_G: U17.10 (G)
- new net SEVEN_SEG_2_A: U25.7 (A)
- new net SEVEN_SEG_2_B: U25.6 (B)
- new net SEVEN_SEG_2_C: U25.4 (C)
- new net SEVEN_SEG_2_D: U25.2 (D)
- new net SEVEN_SEG_2_DP: U25.5 (DP)
- new net SEVEN_SEG_2_E: U25.1 (E)
- new net SEVEN_SEG_2_F: U25.9 (F)
- new net SEVEN_SEG_2_G: U25.10 (G)
- new net SEVEN_SEG_3_A: U26.7 (A)
- new net SEVEN_SEG_3_B: U26.6 (B)
- new net SEVEN_SEG_3_C: U26.4 (C)
- new net SEVEN_SEG_3_D: U26.2 (D)
- new net SEVEN_SEG_3_DP: U26.5 (DP)
- new net SEVEN_SEG_3_E: U26.1 (E)
- new net SEVEN_SEG_3_F: U26.9 (F)
- new net SEVEN_SEG_3_G: U26.10 (G)
- new net SEVEN_SEG_4_A: U27.7 (A)
- new net SEVEN_SEG_4_B: U27.6 (B)
- new net SEVEN_SEG_4_C: U27.4 (C)
- new net SEVEN_SEG_4_D: U27.2 (D)
- new net SEVEN_SEG_4_DP: U27.5 (DP)
- new net SEVEN_SEG_4_E: U27.1 (E)
- new net SEVEN_SEG_4_F: U27.9 (F)
- new net SEVEN_SEG_4_G: U27.10 (G)
Other:
- note added: "TODO: During test check stiffness of ADC supplies, we may need more current delivery here during 10MHz switching especially!"
- note removed: "TODO: Hook up 7 segs"
- note removed: "https://au.element14.com/kingbright/kcpsc04-123/led-alpha-num-10-16mm-green/dp/2449718"
- moved on the sheet: C21, C22, C23, C27, C28, C29, C30, C31, C33, C34, C35, C36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
