File: analog_front_end_v2.kicad_sch (KiCad schematic)
At the start: 208 parts, among them J1 Conn_Coaxial, J3 Conn_01x01_Socket, J4 Conn_01x01_Socket, T1 JTX-4-10T_, U1 ADL5531, U10 PMOD 2x6, U11 LP2985-5.0, U12 LP2985-5.0, U13 ADA4899-1YRDZ, U14 MAX 735, U15 LP2985-2.5, U16 LT5546, U17 KCSA02-123, U18 PAT1220-C-0DB, U19 PAT1220-C-0DB, U2 ADL5531, U20 PAT1220-C-0DB, U21 PAT1220-C-0DB, U22 LP2985-3.3, U23 PMOD 2x6, U24 ADA4899-1YRDZ, U25 KCSA02-123, U26 KCSA02-123, U27 KCSA02-123, U28 LM1117MP-3.3, U3 ADL5531, U4 ADA4899-1YRDZ, U5 ADF4360-9, U6 LT5546, U7 LT5546, U8 ADA4899-1YRDZ, U9 PMOD 2x6

Commit message: Assigning resistor and cap MOC's within the op-amps section
Parts:
- C33, C62, C65, C68, C76, C77, C82, C83: MOC (none) -> 0603YC105JAT2A
- C61, C66, C78, C79: MOC (none) -> 04023A100FAT2A; Tolerance (none) -> 1%
- C63, C64, C70, C71, C86, C87, C91, C92: MOC (none) -> GRT1555C1H201FA02D; Tolerance (none) -> 1%
- L11: value 159n -> 160n; footprint Inductor_SMD:L_1008_2520Metric -> Inductor_SMD:L_0402_1005Metric_Pad0.77x0.64mm_HandSolder; MOC (none) -> MLJ1005WR16JT000; Size (none) -> 0402
- R13, R22, R40, R47: MOC (none) -> TNPW040249K3BEED; Tolerance 1% -> 0.1%
- R14, R23, R48, R49: MOC (none) -> ERA-8AEB753V; Tolerance 1% -> 0.1%
- R15, R20, R38, R39: MOC (none) -> TNPW04024K22BETD; Tolerance 1% -> 0.1%
- R26, R32, R37, R56, R57: MOC (none) -> RC0402FR-07100RL
Other:
- note added: "TODO: Add connectors to Arty-S7 here"
- note added: "TODO: Assign resistor MOC's here"
- moved on the sheet: C1, C5, J1, L1, L2, L3

Commit message: Assign remaining passive MOC's
Parts:
- C40, C41, C55, C60, C72, C73, C74, C75, C81, C85, C88, C89, C90, C93: MOC (none) -> 0402B104K250HI
- R11, R19, R28, R29: MOC (none) -> ERA-2AEB203X
- R16, R24, R50, R52: MOC (none) -> ERA-2AEB822X; Tolerance 1% -> 0.1%
- R17, R27, R54, R55: MOC (none) -> ERA-6AEB2431V; Tolerance 1% -> 0.1%
- R18, R25, R51, R53: MOC (none) -> CPF0402B24R9E; Tolerance 1% -> 0.1%
- R36, R4, R58, R59, R60, R61: MOC (none) -> RC0402FR-07100RL
Other:
- note removed: "TODO: Assign resistor MOC's here"
- moved on the sheet: C21, C22, C23, C42, C43, C44, C45, C46, C47, C48, C49, C50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

Commit message: Remove 7 seg's from schematic/PCB, it is extra unneeded noise
Parts:
- removed C94: 10u_50V, Capacitor_SMD:C_1206_3216Metric, symbol Device:C
- removed C95: 47u_16V, Capacitor_SMD:C_1206_3216Metric, symbol Device:C
- removed U17, U25, U26, U27: KCSA02-123, Display_7Segment:KCSC02-123, symbol Display_Character:KCSA02-123
- removed U28: LM1117MP-3.3, Package_TO_SOT_SMD:SOT-223-3_TabPin2, symbol Regulator_Linear:LM1117MP-3.3
- added U17: PMOD 2x6, Connector_PinHeader_1.00mm:PinHeader_2x06_P1.00mm_Vertical, symbol TheEEView_Global_Lib:PMOD_2x6
- C28, C29: MOC (none) -> CC0402JRNPO9BN101; Tolerance (none) -> 5%
- R7, R8: MOC (none) -> ERA-2AEB49R9X; Tolerance (none) -> 0.1%
- U13, U24, U4, U8: footprint ADA4899-1YRDZ:SOIC127P600X175-9N -> Package_SO:SOIC-8-1EP_3.9x4.9mm_P1.27mm_EP2.29x3mm_ThermalVias
- U16, U6: value LT5546 -> LTC2386-16; footprint (none) -> TheEEView_Footprint_Lib:LTC2386-16
- U7: footprint (none) -> TheEEView_Footprint_Lib:LT5546
Connections:
- net ADC_D1 is gone; now on net ADC_I_CNV-: U9.2
- net ADC_D2 is gone; now on net ADC_I_CLK+: U9.3
- net ADC_D3 is gone; now on net ADC_I_CLK-: U9.4
- net ADC_D4 is gone; now on net ADC_I_DA-: U9.7
- net ADC_D5 is gone; now on net ADC_I_DA+: U9.8
- net ADC_D6 is gone; now on net ADC_I_DCO-: U9.9
- net ADC_D7 is gone; now on net ADC_I_DCO+: U9.10
- net 3.3V_PMOD: now also U17.12, U17.6
- net ADC_I_CNV+: now also U9.1
- net ADC_I_DA+: no longer R57.1, U6.16 (DB+)
- net ADC_I_DA-: no longer R57.2, U6.15 (DB-)
- net ADC_Q_CLK+: now also U23.9
- net ADC_Q_CLK-: now also U23.8
- net ADC_Q_CNV+: now also U23.3
- net ADC_Q_CNV-: now also U23.4
- net ADC_Q_DA+: now also U17.1, U17.3
- net ADC_Q_DA-: now also U17.2, U17.4
- net ADC_Q_DCO+: now also U23.7
- net GND: now also U17.11, U17.5
- net ADC_I_DB+: now reaches U23.1
- net ADC_I_DB+: now also R57.1, U6.16 (DB+)
- net ADC_I_DB-: now reaches U23.2
- net ADC_I_DB-: now also R57.2, U6.15 (DB-)
Other:
- note added: "Arty S7 Connectors"
- note added: "TODO: Connect pin 17 to GND! thermal"
- note added: "TODO: Connect pin 33 to GND! thermal"
- note removed: "101.4 (4 green 7 segments, don't display MHz, redundant)"
- note removed: "Arty S7 Connector"
- note removed: "NOTE: NC D0 as it will be noisy!"
- note removed: "TODO: Add connectors to Arty-S7 here"
- moved on the sheet: C21, L14, L15, R7, R8, U23, U9

Commit message: Remove overly complex I/Q demod and post amplification. Reduce to simply 6x LNA's instead to head towards 0dBm received
Parts:
- R6: MOC (none) -> ERA2AEB241XCopied; Tolerance (none) -> 0.1%
- T1: footprint JTX-4-10T_:JTX410T -> (none)
Connections:
- net GND: no longer C7.2, C8.1, L13.1, U7.3 (IF-)
- new net: C7.2, C8.1, L13.1, U7.3 (IF-)
Other:
- note added: "-93dBm approx signal coming in my office"
- note added: "TODO: Add footprint"
- moved on the sheet: C8
Changed lines of the file:
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@@
 		)
 	)
+	(text "TODO: Add footprint"
+		(exclude_from_sim no)
+		(at 363.474 99.314 0)
+		(effects
+			(font
+				(size 1.27 1.27)
+			)
+		)
+	)
 	(text "PCB: To reduce mutual coupling, the inductors\nshould be placed at right angles to one another. "
 		(exclude_from_sim no)
@@
 		)
 	)
+	(text "-93dBm approx signal coming in my office"
+		(exclude_from_sim no)
+		(at 36.576 34.798 0)
+		(effects
+			(font
+				(size 0.762 0.762)
+			)
+		)
+	)
 	(text "3x20dB fixed gain amps (60dB fixed gain)"
 		(exclude_from_sim no)
@@
 	)
 	(junction
+		(at 356.87 50.8)
+		(diameter 0)
+		(color 0 0 0 0)
+	)
+	(junction
 		(at 596.9 62.23)
 		(diameter 0)
@@
 	)
 	(junction
-		(at 358.14 50.8)
+		(at 347.98 50.8)
 		(diameter 0)
 		(color 0 0 0 0)
@@
 	)
 	(junction
-		(at 358.14 41.91)
-		(diameter 0)
-		(color 0 0 0 0)
-	)
-	(junction
 		(at 609.6 200.66)
 		(diameter 0)
@@
 	)
 	(junction
-		(at 372.11 133.35)
+		(at 356.87 41.91)
 		(diameter 0)
 		(color 0 0 0 0)
 	)
 	(junction
-		(at 541.02 62.23)
+		(at 372.11 133.35)
 		(diameter 0)
 		(color 0 0 0 0)
 	)
 	(junction
-		(at 347.98 50.8)
+		(at 541.02 62.23)
 		(diameter 0)
 		(color 0 0 0 0)
@@
 	(wire
 		(pts
-			(xy 358.14 50.8) (xy 347.98 50.8)
-		)
-		(stroke
-			(width 0)
-			(type default)
-		)
-	)
-	(wire
-		(pts
 			(xy 483.87 213.36) (xy 483.87 214.63)
 		)
@@
 	(wire
 		(pts
-			(xy 351.79 41.91) (xy 358.14 41.91)
+			(xy 351.79 41.91) (xy 356.87 41.91)
 		)
 		(stroke
@@
 	(wire
 		(pts
-			(xy 358.14 41.91) (xy 364.49 41.91)
-		)
-		(stroke
-			(width 0)
-			(type default)
-		)
-	)
-	(wire
-		(pts
 			(xy 453.39 130.81) (xy 457.2 130.81)
 		)
@@
 	(wire
 		(pts
+			(xy 347.98 50.8) (xy 356.87 50.8)
+		)
+		(stroke
+			(width 0)
+			(type default)
+		)
+	)
+	(wire
+		(pts
 			(xy 365.76 114.3) (xy 365.76 115.57)
 		)
@@
 	(wire
 		(pts
-			(xy 358.14 41.91) (xy 358.14 43.18)
+			(xy 356.87 41.91) (xy 356.87 43.18)
 		)
 		(stroke
@@
 	(wire
 		(pts
+			(xy 356.87 41.91) (xy 364.49 41.91)
+		)
+		(stroke
+			(width 0)
+			(type default)
+		)
+	)
+	(wire
+		(pts
 			(xy 146.05 24.13) (xy 151.13 24.13)
 		)
@@
 	(wire
 		(pts
-			(xy 361.95 50.8) (xy 358.14 50.8)
+			(xy 361.95 50.8) (xy 356.87 50.8)
 		)
 		(stroke
@@
 		)
 	)
-	(wire
-		(pts
-			(xy 358.14 50.8) (xy 358.14 60.96)
-		)
-		(stroke
-			(width 0)
-			(type default)
-		)
-	)
 	(label "5V_ADC_150mA"
 		(at 191.77 106.68 0)
@@
 	(symbol
 		(lib_id "Device:C")
-		(at 358.14 46.99 180)
+		(at 356.87 46.99 180)
 		(unit 1)
 		(exclude_from_sim no)
@@
 		(dnp no)
 		(property "Reference" "C8"
-			(at 354.584 45.212 0)
+			(at 353.314 45.212 0)
 			(effects
 				(font
@@
 		)
 		(property "Value" "15.9pF"
-			(at 355.6 46.736 0)
+			(at 354.33 46.736 0)
 			(effects
 				(font
@@
 		)
 		(property "Footprint" "Capacitor_SMD:C_0402_1005Metric"
-			(at 357.1748 43.18 0)
+			(at 355.9048 43.18 0)
 			(effects
 				(font
@@
 		)
 		(property "Datasheet" "~"
-			(at 358.14 46.99 0)
+			(at 356.87 46.99 0)
 			(effects
 				(font
@@
 		)
 		(property "Description" "Unpolarized capacitor"
-			(at 358.14 46.99 0)
+			(at 356.87 46.99 0)
 			(effects
 				(font
@@
 		)
 		(property "Size" "0402"
-			(at 356.616 49.022 0)
+			(at 355.346 49.022 0)
 			(effects
 				(font
@@
 		)
 		(property "MOC" "GRT1555C1H160FA02D"
-			(at 358.14 46.99 0)
+			(at 356.87 46.99 0)
 			(effects
 				(font
@@
 		)
 		(property "Tolerance" "1%"
-			(at 356.616 50.038 0)
+			(at 355.346 50.038 0)
 			(effects
 				(font
@@
 	)
 	(symbol
-		(lib_id "power:GND")
-		(at 358.14 60.96 0)
-		(unit 1)
-		(exclude_from_sim no)
-		(in_bom yes)
-		(on_board yes)
-		(dnp no)
-		(property "Reference" "#PWR026"
-			(at 358.14 67.31 0)
-			(effects
-				(font
-					(size 1.27 1.27)
-				)
-				(hide yes)
-			)
-		)
-		(property "Value" "GND"
-			(at 358.14 64.516 0)
-			(effects
-				(font
-					(size 0.762 0.762)
-				)
-			)
-		)
-		(property "Footprint" ""
-			(at 358.14 60.96 0)
-			(effects
-				(font
-					(size 1.27 1.27)
-				)
-				(hide yes)
-			)
-		)
-		(property "Datasheet" ""
-			(at 358.14 60.96 0)
-			(effects
-				(font
-					(size 1.27 1.27)
-				)
-				(hide yes)
-			)
-		)
-		(property "Description" "Power symbol creates a global label with name \"GND\" , ground"
-			(at 358.14 60.96 0)
-			(effects
-				(font
-					(size 1.27 1.27)
-				)
-				(hide yes)
-			)
-		)
-		(pin "1"
-		)
-		(instances
-			(project "analog_front_end_v2"
-				(path "/6d1f935e-d802-4e58-92ff-681b892e6136"
-					(reference "#PWR026")
-					(unit 1)
-				)
-			)
-		)
-	)
-	(symbol
 		(lib_id "Device:L")
 		(at 93.98 46.99 0)
@@
 			)
 		)
-		(property "Footprint" "JTX-4-10T_:JTX410T"
+		(property "Footprint" ""
 			(at 341.63 88.9 0)
 			(effects
@@
 			)
 		)
-		(property "MOC" ""
+		(property "MOC" "ERA2AEB241XCopied"
 			(at 396.24 92.71 90)
 			(effects
@@
 			)
 		)
-		(property "Tolerance" ""
-			(at 398.018 92.71 90)
+		(property "Tolerance" "0.1%"
+			(at 398.526 92.964 0)
 			(effects
 				(font
 					(size 0.4572 0.4572)
 				)
-				(hide yes)
 			)
 		)

Commit message: Shrink down all schematic connections for a simpler painting
Parts:
- removed C41, C55, C60, C72, C73, C74, C75, C81, C85, C88, C89, C90, C93: 0.1uF, Capacitor_SMD:C_0402_1005Metric, symbol Device:C
- removed C50: 82pF_16V, Capacitor_SMD:C_0402_1005Metric, symbol Device:C
- removed C51: 10u_16V, Capacitor_SMD:C_1206_3216Metric, symbol Device:C_Polarized_US
- removed C52: 10n_25V, Capacitor_SMD:C_0402_1005Metric, symbol Device:C
- removed C53: 10u_50V, Capacitor_SMD:C_1206_3216Metric, symbol Device:C
- removed C54, C56, C57, C67, C69: 10u_16V, Capacitor_SMD:C_0805_2012Metric, symbol Device:C
- removed C58, C59, C80, C84: 100n_25V, Capacitor_SMD:C_0402_1005Metric, symbol Device:C
- removed C61, C66, C78, C79: 10p_50V, Capacitor_SMD:C_0402_1005Metric, symbol Device:C
- removed C62, C65, C68, C76, C77, C82, C83: 1u_16V, Capacitor_SMD:C_0402_1005Metric, symbol Device:C
- removed C63, C64, C70, C71, C86, C87, C91, C92: 200p_50V, Capacitor_SMD:C_0402_1005Metric, symbol Device:C
- removed D1: 1N5817, Diode_THT:D_DO-41_SOD81_P10.16mm_Horizontal, symbol Diode:1N5817
- removed D4: LED, LED_SMD:LED_0603_1608Metric, symbol Device:LED
- removed L18: 10u, TheEEView_Footprint_Lib:SRU1028A-100Y, symbol Device:L
- removed R11, R19, R28, R29: 20kR, Resistor_SMD:R_0402_1005Metric, symbol Device:R
- removed R13, R22, R40, R47: 49k3R, Resistor_SMD:R_0402_1005Metric, symbol Device:R
- removed R14, R23, R48, R49: 75kR, Resistor_SMD:R_0402_1005Metric, symbol Device:R
- removed R15, R20, R38, R39: 4k22R, Resistor_SMD:R_0402_1005Metric, symbol Device:R
- removed R16, R24, R50, R52: 8k2R, Resistor_SMD:R_0402_1005Metric, symbol Device:R
- removed R17, R27, R54, R55: 2k43R, Resistor_SMD:R_0402_1005Metric, symbol Device:R
- removed R18, R25, R51, R53: 24R9, Resistor_SMD:R_0402_1005Metric, symbol Device:R
- removed R21: 50R, Resistor_SMD:R_0603_1608Metric, symbol Device:R
- removed R26, R32, R36, R37, R4, R56, R57, R58, R59, R60, R61: 100R, Resistor_SMD:R_0402_1005Metric, symbol Device:R
- removed R33: 130k, Resistor_SMD:R_0402_1005Metric, symbol Device:R
- removed R34: 300k, Resistor_SMD:R_0402_1005Metric, symbol Device:R
- removed R35, R5: 0R, Resistor_SMD:R_0402_1005Metric, symbol Device:R
- removed U13, U24, U4, U8: ADA4899-1YRDZ, Package_SO:SOIC-8-1EP_3.9x4.9mm_P1.27mm_EP2.29x3mm_ThermalVias, symbol ADA4899-1YRDZ:ADA4899-1YRDZ
- removed U14: MAX 735, Package_SO:SOIC-8_5.3x5.3mm_P1.27mm, symbol TheEEView_Global_Lib:MAX735
- removed U15: LP2985-2.5, Package_TO_SOT_SMD:SOT-23-5, symbol Regulator_Linear:LP2985-2.5
- removed U16, U6: LTC2386-16, TheEEView_Footprint_Lib:LTC2386-16, symbol TheEEView_Global_Lib:LTC2386
- removed U17: PMOD 2x6, Connector_PinHeader_1.00mm:PinHeader_2x06_P1.00mm_Vertical, symbol TheEEView_Global_Lib:PMOD_2x6
- removed U22: LP2985-3.3, Package_TO_SOT_SMD:SOT-23-5, symbol Regulator_Linear:LP2985-3.3
- removed U7: LT5546, TheEEView_Footprint_Lib:LT5546, symbol TheEEView_Global_Lib:LT5546EUF
- added C41: 47u_16V, Capacitor_Tantalum_SMD:CP_EIA-6032-15_Kemet-U, symbol Device:C_Polarized_US
- added D1: LED, LED_SMD:LED_0603_1608Metric, symbol Device:LED
- added TP1, TP2, TP3: TestPoint, TestPoint:TestPoint_Pad_D1.0mm, symbol Connector:TestPoint
- added U13, U24, U7: PAT1220-C-0DB, RF_Converter:RF_Attenuator_Susumu_PAT1220, symbol RF:PAT1220-C-0DB
- added U14: LP2985-5.0, Package_TO_SOT_SMD:SOT-23-5, symbol Regulator_Linear:LP2985-5.0
- added U22, U4, U8: ADL5531, TheEEView_Footprint_Lib:ADL5531, symbol TheEEView_Global_Lib:ADL5531
- added U6: MCP33131, symbol TheEEView_Global_Lib:MCP33131
- C21: value 10u_50V -> 1u_16V; footprint Capacitor_SMD:C_1206_3216Metric -> Capacitor_SMD:C_0603_1608Metric; MOC CL31A106KBHNNNE -> 0603YC105JAT2A; Size 1206 -> 0603; Tolerance 10% -> 5%
- C22: value 10n_25V -> 1n_50V; MOC GRM1555C1E103JE01J -> GRM1555C1H102JA01D
- C23, C38: value 10u_16V -> 10n_25V; footprint Capacitor_SMD:C_0805_2012Metric -> Capacitor_SMD:C_0402_1005Metric; MOC CL21B106KOQNNNE -> GRM1555C1E103JE01J; Size 0805 -> 0402; Tolerance 10% -> 5%
- C24: value 1u_16V -> 10n_25V; footprint Capacitor_SMD:C_0603_1608Metric -> Capacitor_SMD:C_0402_1005Metric; MOC 0603YC105JAT2A -> GRM1555C1E103JE01J; Size 0603 -> 0402
- C25: value 1n_50V -> 1u_16V; footprint Capacitor_SMD:C_0402_1005Metric -> Capacitor_SMD:C_0603_1608Metric; MOC GRM1555C1H102JA01D -> 0603YC105JAT2A; Size 0402 -> 0603
- C30: value 1p5F -> 10n_25V; MOC CBR04C159B1GAC -> GRM1555C1E103JE01J; Tolerance 0.1pF -> 5%
- C31: value 1p8F -> 10n_25V; MOC QSCF500Q1R8B1GV001T -> GRM1555C1E103JE01J; Tolerance 0.1pF -> 5%
- C33: footprint Capacitor_SMD:C_0402_1005Metric -> Capacitor_SMD:C_0603_1608Metric; Size 0402 -> 0603; Tolerance (none) -> 5%
- C36: value 10u_16V -> 10u_50V; footprint Capacitor_SMD:C_0805_2012Metric -> Capacitor_SMD:C_1206_3216Metric; MOC CL21B106KOQNNNE -> CL31A106KBHNNNE; Size 0805 -> 1206
- C40: value 0.1uF -> 10u_16V; footprint Capacitor_SMD:C_0402_1005Metric -> Capacitor_SMD:C_0805_2012Metric; MOC 0402B104K250HI -> CL21B106KOQNNNE; Size 0402 -> 0805
- C49: value 10u_16V -> 47u_16V; footprint Capacitor_SMD:C_1206_3216Metric -> Capacitor_Tantalum_SMD:CP_EIA-6032-15_Kemet-U; MOC TAJA106K016RNJ -> TAJC476K016RNJ; Size 1206 -> 2312
- C6: value 220pF -> 1n_50V; MOC GRT1555C1E221FA02D -> GRM1555C1H102JA01D; Tolerance 1% -> 5%
- C7, C8: value 15.9pF -> 10n_25V; MOC GRT1555C1H160FA02D -> GRM1555C1E103JE01J; Tolerance 1% -> 5%
- L11, L13: value 160n -> 470n; footprint Inductor_SMD:L_0402_1005Metric_Pad0.77x0.64mm_HandSolder -> Inductor_SMD:L_1008_2520Metric; MOC MLJ1005WR16JT000 -> 1008CS-471XGRC; Size 0402 -> 1008
- R2: value 20kR -> 150R; footprint Resistor_SMD:R_0402_1005Metric -> Resistor_SMD:R_0603_1608Metric; MOC RC0402FR-0720KL -> RC0805FR-07150RL; Size 0402 -> 0603
Connections:
- net DEMOD_I+ is gone; now on net 5V_LNA2: C33.1
- net 5V_ADC: now also C49.1; no longer C36.2, C40.2
- net GND: now also C21.2, C22.2, C23.2, C30.2, C33.2, C6.2, C7.2, C41.2, D1.1 (K), TP1.1, TP2.1, TP3.1, U13.3, U14.2 (GND), U22.9 (EP), U24.3, U4.9 (EP), U7.3, U8.9 (EP); no longer C21.1, C22.1, C23.1, C24.1, C30.1, C31.1, L12.2, L13.2
- net VIN: now also C36.2, U14.1 (VIN), U14.3 (ON/~{OFF}); no longer C21.2
- net at R2.1: now also D1.2 (A)
- net at R1.1: now also C40.2, U14.5 (VOUT); no longer C23.2
- net at C8.2: now also U7.1; no longer L11.2
- net at U21.2: now also U4.2 (RFIN); no longer C6.1
- net 2V5_ADC: no longer names the net of C38.2
- net 2V5_ADC: now also U14.4 (BP)
- net 3.3V_IQ_DEMOD renamed 5V_LNA2
- net 5V_LNA2: now also C21.1, C23.1, C30.1, C7.1, L11.2, L12.2, L13.2, C41.1; no longer C24.2, C26.1
- net 5V_LNA renamed 5V_LNA1
- net ADC_I_CLK+: no longer names the net of U9.3
- net ADC_I_CLK-: no longer names the net of U9.4
- net ADC_I_CNV+: no longer names the net of U9.1
- net ADC_I_CNV-: no longer names the net of U9.2
- net ADC_I_DA+: no longer names the net of U9.8
- net ADC_I_DA-: no longer names the net of U9.7
- net ADC_I_DB+: no longer names the net of U23.1
- net ADC_I_DB-: no longer names the net of U23.2
- net ADC_I_DCO+: no longer names the net of U9.10
- net ADC_I_DCO-: no longer names the net of U9.9
- net ADC_Q_CLK+: no longer names the net of U23.9
- net ADC_Q_CLK-: no longer names the net of U23.8
- net ADC_Q_CNV+: no longer names the net of U23.3
- net ADC_Q_CNV-: no longer names the net of U23.4
- net ADC_Q_DCO+: no longer names the net of U23.7
- net DEMOD_IF_DET: no longer names the net of C31.2
- net DEMOD_IF_DET: now also U24.1
- net DEMOD_VCTRL: no longer names the net of U23.10
- new net: C31.1, L13.1, U22.7 (RFOUT)
- new net: C24.2, U13.1
- new net: U13.2, U22.2 (RFIN)
- new net: C22.1, U8.5 (CLIN)
- new net: C8.1, L11.1, U4.7 (RFOUT)
- new net: U7.2, U8.2 (RFIN)
- new net: C24.1, L12.1, U8.7 (RFOUT)
- new net: C6.1, U4.5 (CLIN)
- new net: C26.1, U22.5 (CLIN)
- no-connect marks 19 -> 34
Other:
- note added: "6x20dB fixed gain amps (120dB fixed gain)"
- note added: "GND Testpoints"
- note added: "TODO: Shift up AC wave to use full dynamic range"
- note removed: "2x 16-bit ADC Front End for I/Q"
- note removed: "3x20dB fixed gain amps (60dB fixed gain)"
- note removed: "GND Testpoint"
- note removed: "I/Q Demod"
- note removed: "IF low pass filter"
- note removed: "PWM Output from FPGA"
- note removed: "TODO: Connect pin 17 to GND! thermal"
- note removed: "TODO: Connect pin 33 to GND! thermal"
- moved on the sheet: C10, C11, C12, C13, C14, C15, C16, C17, C18, C19, C2, C20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

Commit message: Reduce LNA total gain down to 100dB, should be enough to support -93dBm received signals in Melbourne with plenty of signal at the ADC.
Parts:
- removed C26: 1n_50V, Capacitor_SMD:C_0402_1005Metric, symbol Device:C
- removed C30, C31: 10n_25V, Capacitor_SMD:C_0402_1005Metric, symbol Device:C
- removed C33: 1u_16V, Capacitor_SMD:C_0603_1608Metric, symbol Device:C
- removed L13: 470n, Inductor_SMD:L_1008_2520Metric, symbol Device:L
- removed U22: ADL5531, TheEEView_Footprint_Lib:ADL5531, symbol TheEEView_Global_Lib:ADL5531
- removed U24: PAT1220-C-0DB, RF_Converter:RF_Attenuator_Susumu_PAT1220, symbol RF:PAT1220-C-0DB
Connections:
- no-connect marks 34 -> 29
Other:
- note added: "5x20dB fixed gain amps (100dB fixed gain)"
- note added: "Goals: 1. Support from -95dBm received signal 2. 50 ohm impedance 3. Minimize parasitics (inc trace resistance) as much as possible in layout to lock on center freq 4. Via stiching to ground around RF traces 5. Short traces with minimal direction changes"
- note added: "TODO: Shift up AC wave by 1V to use full dynamic range Use an RF bias tee for this: RF In (50Ω) ----[L (RFC)]----+---- RF Out (50Ω) to ADC | [C] | +1V DC"
- note removed: "6x20dB fixed gain amps (120dB fixed gain)"
- note removed: "Goals: 1. 50 ohm impedance 2. Minimize parasitics (inc trace resistance) as much as possible in layout to lock on center freq 3. Via stiching to ground around RF traces 4. Short traces with minimal direction changes"
- note removed: "TODO: Shift up AC wave to use full dynamic range"
- moved on the sheet: C27, C28, C29, C32, C34, C35, C37, C39, L14, L15, L6, L7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

Commit message: Latest changes to add in a new diffamp and simplify the schematic for readability
Parts:
- removed C27: 1n_50V, Capacitor_SMD:C_0402_1005Metric, symbol Device:C
- removed C28, C29: 100p_50V, Capacitor_SMD:C_0402_1005Metric, symbol Device:C
- removed C32: 22n_25V_COG, Capacitor_SMD:C_0402_1005Metric, symbol Device:C
- removed C34: 10u_16V, Capacitor_SMD:C_0805_2012Metric, symbol Device:C
- removed C35: 56p_50V, Capacitor_SMD:C_0402_1005Metric, symbol Device:C
- removed C37: 2.2n_50V, Capacitor_SMD:C_0603_1608Metric, symbol Device:C
- removed C39: 150p_150V, Capacitor_SMD:C_0402_1005Metric, symbol Device:C
- removed L14, L15: 72n, Inductor_SMD:L_0402_1005Metric, symbol Device:L
- removed L6, L7: 250n, Inductor_SMD:L_0402_1005Metric, symbol Device:L
- removed R10, R9: 0R, Resistor_SMD:R_0402_1005Metric, symbol Device:R
- removed R12: 4.7kR, Resistor_SMD:R_0402_1005Metric, symbol Device:R
- removed R41: 12kR, Resistor_SMD:R_0402_1005Metric, symbol Device:R
- removed R42: 5.6kR, Resistor_SMD:R_0402_1005Metric, symbol Device:R
- removed R43, R44: 470R, Resistor_SMD:R_0402_1005Metric, symbol Device:R
- removed R8: 49R9, Resistor_SMD:R_0402_1005Metric, symbol Device:R
- removed T1: JTX-4-10T_, symbol JTX-4-10T_:JTX-4-10T_
- removed TP1, TP2, TP3: TestPoint, TestPoint:TestPoint_Pad_D1.0mm, symbol Connector:TestPoint
- removed U10: PMOD 2x6, Connector_PinHeader_1.00mm:PinHeader_2x06_P1.00mm_Vertical, symbol TheEEView_Global_Lib:PMOD_2x6
- removed U5: ADF4360-9, TheEEView_Footprint_Lib:ADF4360-9, symbol TheEEView_Global_Lib:ADF4360-9
- added R3: 357, symbol Device:R
- added R4: 22.6, symbol Device:R
- added R5: 127, symbol Device:R
- added U5: LMH5401, symbol TheEEView_Global_Lib:LMH4501
- R6: value 240R -> 66.5; footprint Resistor_SMD:R_0402_1005Metric -> (none); MOC ERA2AEB241XCopied -> ERA-2AEB3570X
- R7: value 49R9 -> 127; footprint Resistor_SMD:R_0402_1005Metric -> (none); MOC ERA-2AEB49R9X -> ERA-2AEB3570X; now fitted
Connections:
- net GND: now also R3.1; no longer R7.2
- net at U13.2: now also R3.2, R4.1
- net LO+: no longer names the net of R6.2
- net LO-: no longer names the net of R6.1
- new net: R4.2, R5.2, U5.5 (IN-)
- no-connect marks 29 -> 25
Other:
- note added: "-93dBm approx signal coming into my home office"
- note added: "GND Testpoint"
- note added: "Single Ended -> Differential"
- note added: "TODO: Check stiffness of these, we may need more current delivery, during 10MHz switching especially!"
- note added: "TODO: Implement a MAX2606 here"
- note added: "VCO"
- note removed: "-93dBm approx signal coming in my office"
- note removed: "GND Testpoints"
- note removed: "Note: L6 and L7 value sets the PLL centre output frequency 250nH should get the 88MHz to 100MHz range roughly"
- note removed: "PCB: To reduce mutual coupling, the inductors should be placed at right angles to one another."
- note removed: "PLL"
- note removed: "TODO: Add footprint"
- note removed: "TODO: During test check stiffness of ADC supplies, we may need more current delivery here during 10MHz switching especially!"
- moved on the sheet: C1, C10, C11, C12, C13, C14, C15, C16, C17, C18, C19, C2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
