File: analog_front_end_v2.kicad_sch (KiCad schematic)
At the start: 83 parts, among them J1 Conn_Coaxial, J3 Conn_01x01_Socket, J4 Conn_01x01_Socket, U1 ADL5531, U11 LP2985-5.0, U12 LP2985-5.0, U13 PAT1220-C-0DB, U14 LP2985-5.0, U18 PAT1220-C-0DB, U19 PAT1220-C-0DB, U2 ADL5531, U20 PAT1220-C-0DB, U21 PAT1220-C-0DB, U23 PMOD 2x6, U3 ADL5531, U4 ADL5531, U5 LMH5401, U6 MCP33131, U7 PAT1220-C-0DB, U8 ADL5531, U9 PMOD 2x6

Commit message: Fully connected schematic
Parts:
- removed R31: 0R, Resistor_SMD:R_0402_1005Metric, symbol Device:R
- removed U12: LP2985-5.0, Package_TO_SOT_SMD:SOT-23-5, symbol Regulator_Linear:LP2985-5.0
- removed U23: PMOD 2x6, Connector_PinHeader_1.00mm:PinHeader_2x06_P1.00mm_Vertical, symbol TheEEView_Global_Lib:PMOD_2x6
- removed U5: LMH5401, symbol TheEEView_Global_Lib:LMH4501
- added C26: 1u_16V, Capacitor_SMD:C_0603_1608Metric, symbol Device:C
- added C27, C28: 100n_25V, Capacitor_SMD:C_0402_1005Metric, symbol Device:C
- added C29: 1n_50V, Capacitor_SMD:C_0402_1005Metric, symbol Device:C
- added C30: 10u_50V, Capacitor_SMD:C_1206_3216Metric, symbol Device:C
- added C31, C50: 10n_25V, Capacitor_SMD:C_0402_1005Metric, symbol Device:C
- added C32: 10u_16V, Capacitor_SMD:C_0805_2012Metric, symbol Device:C
- added C33: 47u_16V, Capacitor_Tantalum_SMD:CP_EIA-6032-15_Kemet-U, symbol Device:C_Polarized_US
- added C34, C35, C37, C39: 5p1_50V, Capacitor_SMD:C_0402_1005Metric, symbol Device:C
- added L13: 100n, Inductor_SMD:L_0402_1005Metric, symbol Device:L
- added L6: 10n, Inductor_SMD:L_0805_2012Metric, symbol Device:L
- added L7: 390n, Inductor_SMD:L_0805_2012Metric, symbol Device:L
- added R10, R8, R9: 3.3k, symbol Device:R
- added U10: MAX6002, Package_TO_SOT_SMD:SOT-23, symbol Reference_Voltage:MAX6002
- added U12: MAX2606, symbol TheEEView_Global_Lib:MAX2606
- added U15, U16: BFP540ESD, symbol TheEEView_Global_Lib:BFP540ESD
- added U17: LP2985-3.3, Package_TO_SOT_SMD:SOT-23-5, symbol Regulator_Linear:LP2985-3.3
- added U5: LP2985-1.8, Package_TO_SOT_SMD:SOT-23-5, symbol Regulator_Linear:LP2985-1.8
- R3: value 357 -> 100; MOC ERA-2AEB3570X -> RC0402FR-07100RL; Tolerance 0.1% -> 1%
- R4: value 22.6 -> 0R; footprint (none) -> Resistor_SMD:R_0402_1005Metric; MOC ERA-2AEB3570X -> MCMR04X000 PTL; Tolerance 0.1% -> 1%
- R5: value 127 -> 100; MOC ERA-2AEB3570X -> RC0402FR-07100RL; Tolerance 0.1% -> 1%
- R6: value 66.5 -> 100; MOC ERA-2AEB3570X -> RC0402FR-07100RL; Tolerance 0.1% -> 1%
- R7: value 127 -> 0R; footprint (none) -> Resistor_SMD:R_0402_1005Metric; MOC ERA-2AEB3570X -> MCMR04X000 PTL; Tolerance 0.1% -> 1%
Connections:
- net 5V_ADC: no longer C49.1
- net GND: now also U6.4 (AIN-), U6.5 (GND), C27.2, C28.2, C29.1, C30.1, C31.1, C33.2, C50.2, L13.1, L7.1, U10.3 (GND), U12.2 (GND), U17.2 (GND), U5.2 (GND); no longer R3.1
- net VIN: now also C30.2, U17.1 (VIN), U17.3 (ON/~{OFF}), U5.1 (VIN), U5.3 (ON/~{OFF})
- net 1V8: now reaches R4.2
- net 1V8: now also U6.2 (AVDD), C27.1, C33.1; no longer R5.2
- net at R6.1: now also U12.4 (OUT-)
- net 3V3: now reaches R6.2
- net 3V3: now also C49.1, R5.2, R7.2, U6.10 (DVIO), C28.1, C37.2, C50.1, R10.1, R8.1, R9.1, U10.1 (IN), U12.5 (VCC)
- net at R5.1: now also U12.6 (OUT+)
- net ADC_SDI: now reaches U9.1
- net ADC_SDI: now also U6.9 (SDI)
- net ADC_SDO: now reaches U9.2
- net ADC_SDO: now also U6.7 (SDO)
- net ADC_SCLK: now reaches U9.3
- net ADC_SCLK: now also U6.8 (SCLK)
- net ADC_CONVST: now reaches U9.9
- net ADC_CONVST: now also U6.6 (CONVST)
- net at C46.2: now also U17.4 (BP)
- net at C47.2: now also R7.1, U17.5 (VOUT)
- net ADC_VREF: now reaches U6.1 (Vref)
- net ADC_VREF: now also U10.2 (OUT)
- net at U6.3 (AIN+): now also C26.2, L6.1
- new net: C39.2, R9.2, U15.1 (B)
- new net: C31.2, U5.4 (BP)
- new net: C32.2, R4.1, U5.5 (VOUT)
- new net: C34.2, U13.2
- new net: L7.2, U12.1 (IND)
- new net: C35.2, R8.2, U16.1 (B)
- new net: L13.2, U16.2 (E), U16.4 (E)
- new net: U15.2 (E), U15.4 (E), U16.3 (C)
- new net: C34.1, C35.1
- new net: L6.2, R3.2
- new net: C37.1, C39.1
- new net: C26.1, R10.2, U15.3 (C)
- new net: C29.2, U12.3 (TUNE)
- new net 1V: R3.1
Other:
- note added: "ADC"
- note added: "Arty S7 Connector"
- note added: "Cascode mixer for 96MHz to 106MHz band"
- note added: "Inductor has Q close to 40 around 100MHz"
- note removed: "Arty S7 Connectors"
- note removed: "NOTE: OFUF NC as not enough pins on PMOD!"
- note removed: "Single Ended -> Differential"
- note removed: "TODO: Implement a MAX2606 here"
- note removed: "TODO: Shift up AC wave by 1V to use full dynamic range Use an RF bias tee for this: RF In (50Ω) ----[L (RFC)]----+---- RF Out (50Ω) to ADC | [C] | +1V DC"
- moved on the sheet: C1, C10, C11, C12, C13, C14, C15, C16, C17, C18, C19, C2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
