File: analog_front_end_v2.kicad_pcb (KiCad board)
At the start: 4 copper layers, 253 parts, among them J1 Conn_Coaxial, J3 Conn_01x01_Socket, J4 Conn_01x01_Socket, U1 ADL5531, U10 PMOD 2x6, U11 LP2985-5.0, U12 LP2985-5.0, U13 ADA4899-1YRDZ, U13 LT1363, U14 MAX 735, U15 LP2985-2.5, U16 LTC2386-16, U16 MAX889SESA, U17 PMOD 2x6, U18 PAT1220-C-0DB, U19 PAT1220-C-0DB, U2 ADL5531, U20 PAT1220-C-0DB, U21 PAT1220-C-0DB, U22 LP2985-3.3, U23 PMOD 2x6, U24 ADA4899-1YRDZ, U3 ADL5531, U4 ADA4899-1YRDZ, U4 PE4140B-Z, U5 ADF4360-9, U6 LTC2386-16, U7 LT5546, U7 THS4551, U8 ADA4899-1YRDZ, U8 LT1363, U9 PMOD 2x6

Commit message: Use consistent 0.6x0.3mm vias and tracing cleanups
Parts:
- removed the C33 at (93.1, 74.7)
- removed D2: LED, LED_SMD:LED_0603_1608Metric
- removed the L11 at (96.6, 100.1)
- removed the L11 at (148.3, 42.4)
- removed the L13 at (87.6, 99.5)
- removed the R10 at (79.7, 76.2)
- removed the R10 at (143.8, 36.5)
- removed the R15 at (78.7, 84.0)
- removed R45: 150R, Resistor_SMD:R_0603_1608Metric
- added C21: 1u_16V, Capacitor_SMD:C_0603_1608Metric, F.Cu at (108.0, 34.3)
- added C22: 1n_50V, Capacitor_SMD:C_0402_1005Metric, F.Cu at (137.6, 78.9)
- added C24: 10n_25V, Capacitor_SMD:C_0402_1005Metric, F.Cu at (121.9, 40.5)
- added C26: 1n_50V, Capacitor_SMD:C_0402_1005Metric, F.Cu at (140.5, 75.0)
- added C26: 1u_16V, Capacitor_SMD:C_0603_1608Metric, F.Cu at (140.4, 46.3)
- added C27: 100n_25V, Capacitor_SMD:C_0402_1005Metric, F.Cu at (141.4, 44.5)
- added C28: 100n_25V, Capacitor_SMD:C_0402_1005Metric, F.Cu at (147.8, 43.1)
- added C29: 1n_50V, Capacitor_SMD:C_0402_1005Metric, F.Cu at (122.7, 48.3)
- added C30: 10n_25V, Capacitor_SMD:C_0402_1005Metric, F.Cu at (140.5, 76.9)
- added C30: 10u_50V, Capacitor_SMD:C_1206_3216Metric, F.Cu at (140.4, 18.7)
- added C31: 10n_25V, Capacitor_SMD:C_0402_1005Metric, F.Cu at (140.5, 78.9)
- added C31: 10n_25V, Capacitor_SMD:C_0402_1005Metric, F.Cu at (139.5, 24.8)
- added C32: 10u_16V, Capacitor_SMD:C_0805_2012Metric, F.Cu at (142.8, 25.3)
- added C33: 1u_16V, Capacitor_SMD:C_0603_1608Metric, F.Cu at (143.9, 89.5)
- added C33: 47u_16V, Capacitor_Tantalum_SMD:CP_EIA-6032-15_Kemet-U, F.Cu at (145.4, 29.3)
- added C34: 5p1_50V, Capacitor_SMD:C_0402_1005Metric, F.Cu at (127.4, 40.5)
- added C35: 5p1_50V, Capacitor_SMD:C_0402_1005Metric, F.Cu at (129.4, 40.5)
- added C36: 10u_50V, Capacitor_SMD:C_1206_3216Metric, F.Cu at (112.0, 18.7)
- added C38: 10n_25V, Capacitor_SMD:C_0402_1005Metric, F.Cu at (111.1, 24.8)
- added C39: 5p1_50V, Capacitor_SMD:C_0402_1005Metric, F.Cu at (130.6, 44.2)
- added C40: 10u_16V, Capacitor_SMD:C_0805_2012Metric, F.Cu at (114.4, 25.3)
- added C41: 47u_16V, Capacitor_Tantalum_SMD:CP_EIA-6032-15_Kemet-U, F.Cu at (117.0, 29.5)
- added C45: 10u_50V, Capacitor_SMD:C_1206_3216Metric, F.Cu at (128.0, 18.7)
- added C47: 10u_16V, Capacitor_SMD:C_0805_2012Metric, F.Cu at (130.4, 25.3)
- added C49: 47u_16V, Capacitor_Tantalum_SMD:CP_EIA-6032-15_Kemet-U, F.Cu at (132.9, 29.5)
- added C49: 47u_16V, Capacitor_Tantalum_SMD:CP_EIA-6032-15_Kemet-U, F.Cu at (118.5, 71.1)
- added C50: 10n_25V, Capacitor_SMD:C_0402_1005Metric, F.Cu at (128.0, 47.3)
- added C51: 100n_25V, Capacitor_SMD:C_0402_1005Metric, F.Cu at (121.5, 48.3)
- added C52: 100n_25V, Capacitor_SMD:C_0402_1005Metric, F.Cu at (139.6, 42.0)
- added C7: 10n_25V, Capacitor_SMD:C_0402_1005Metric, F.Cu at (107.7, 35.7)
- added D1: LED, LED_SMD:LED_0603_1608Metric, F.Cu at (120.8, 77.4)
- added D4: LED, LED_SMD:LED_0603_1608Metric, F.Cu at (152.1, 67.6)
- added L11: 470n, Inductor_SMD:L_1008_2520Metric, F.Cu at (108.3, 37.8)
- added L13: 100n, Inductor_SMD:L_0402_1005Metric, F.Cu at (132.1, 42.4)
- added L13: 470n, Inductor_SMD:L_1008_2520Metric, F.Cu at (144.4, 81.4)
- added L6: 10n, Inductor_SMD:L_0805_2012Metric, F.Cu at (140.1, 48.1)
- added L7: 390n, Inductor_SMD:L_0603_1608Metric, F.Cu at (125.0, 45.0)
- added R1: 0R, Resistor_SMD:R_0402_1005Metric, F.Cu at (114.0, 26.9)
- added R10: 3.3k, Resistor_SMD:R_0402_1005Metric, F.Cu at (138.3, 45.0)
- added R12: 150R, Resistor_SMD:R_0603_1608Metric, F.Cu at (152.1, 70.2)
- added R2: 150R, Resistor_SMD:R_0603_1608Metric, F.Cu at (124.8, 77.4)
- added R3: 100, Resistor_SMD:R_0402_1005Metric, F.Cu at (137.7, 47.6)
- added R4: 0R, Resistor_SMD:R_0402_1005Metric, F.Cu at (142.4, 26.9)
- added R5: 100, Resistor_SMD:R_0402_1005Metric, F.Cu at (129.1, 47.3)
- added R6: 100, Resistor_SMD:R_0402_1005Metric, F.Cu at (128.0, 49.3)
- added R7: 0R, Resistor_SMD:R_0402_1005Metric, F.Cu at (130.0, 26.9)
- added R8: 3.3k, Resistor_SMD:R_0402_1005Metric, F.Cu at (132.1, 40.0)
- added R9: 3.3k, Resistor_SMD:R_0402_1005Metric, F.Cu at (132.2, 44.7)
- added U10: MAX6002, Package_TO_SOT_SMD:SOT-23, F.Cu at (142.2, 41.5)
- added U13: PAT1220-C-0DB, RF_Converter:RF_Attenuator_Susumu_PAT1220, F.Cu at (124.6, 41.1)
- added U14: LP2985-5.0, Package_TO_SOT_SMD:SOT-23-5, F.Cu at (112.5, 22.1)
- added U16: BFP540ESD, Package_TO_SOT_SMD:SOT-343_SC-70-4_Handsoldering, F.Cu at (135.3, 41.2)
- added U17: LP2985-3.3, Package_TO_SOT_SMD:SOT-23-5, F.Cu at (128.5, 22.1)
- added U22: ADL5531, TheEEView_Footprint_Lib:ADL5531, F.Cu at (153.3, 79.1)
- added U24: PAT1220-C-0DB, RF_Converter:RF_Attenuator_Susumu_PAT1220, F.Cu at (149.1, 81.3)
- added U6: MCP33131, Package_SO:MSOP-10_3x3mm_P0.5mm, F.Cu at (145.2, 45.5)
- added U8: ADL5531, TheEEView_Footprint_Lib:ADL5531, F.Cu at (118.5, 40.8)
- C23: value 10u_16V -> 10n_25V; footprint Capacitor_SMD:C_0805_2012Metric -> Capacitor_SMD:C_0402_1005Metric
- C25: value 1n_50V -> 1u_16V; footprint Capacitor_SMD:C_0402_1005Metric -> Capacitor_SMD:C_0603_1608Metric
- C37: value 2.2n_50V -> 5p1_50V; footprint Capacitor_SMD:C_0603_1608Metric -> Capacitor_SMD:C_0402_1005Metric
- C6: value 220pF -> 1n_50V
- C8: value 15.9pF -> 10n_25V
- J3, J4: footprint Connector_PinSocket_1.27mm:PinSocket_1x01_P1.27mm_Vertical -> Connector:Banana_Jack_1Pin
- R11: value 20kR -> 100
- U12: value LP2985-5.0 -> MAX2606; footprint Package_TO_SOT_SMD:SOT-23-5 -> Package_TO_SOT_SMD:SOT-23-6
- U15: value LP2985-2.5 -> BFP540ESD; footprint Package_TO_SOT_SMD:SOT-23-5 -> Package_TO_SOT_SMD:SOT-343_SC-70-4_Handsoldering
- U4: value ADA4899-1YRDZ -> ADL5531; footprint Package_SO:SOIC-8-1EP_3.9x4.9mm_P1.27mm_EP2.29x3mm_ThermalVias -> TheEEView_Footprint_Lib:ADL5531
- U5: value ADF4360-9 -> LP2985-1.8; footprint TheEEView_Footprint_Lib:ADF4360-9 -> Package_TO_SOT_SMD:SOT-23-5
- U7: value LT5546 -> PAT1220-C-0DB; footprint TheEEView_Footprint_Lib:LT5546 -> RF_Converter:RF_Attenuator_Susumu_PAT1220
- moved R13 140.4 mm to (214.0, 32.3)
- moved C30 107.2 mm to (220.0, 44.2)
- moved C31 107.2 mm to (221.3, 44.5)
- moved C32 107.2 mm to (213.4, 43.7)
- moved C56 107.2 mm to (216.9, 44.1)
- moved R14 107.2 mm to (227.4, 51.3)
- moved R19 107.2 mm to (217.7, 41.6)
- moved U16 107.2 mm to (216.8, 50.3)
- moved R20 107.2 mm to (217.7, 40.4)
- moved TP22 107.2 mm to (224.0, 47.8)
- moved U4 107.2 mm to (223.8, 38.5)
- moved U7 107.2 mm to (218.0, 43.7)
- moved C33 107.2 mm to (215.9, 43.2)
- moved R18 107.2 mm to (215.4, 47.0)
- moved U22 100.4 mm to (166.4, 53.8)
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Connections:
- C10 pad 1: 5V_LNA -> 5V_LNA1 (x2)
- C11 pad 1: 5V_LNA -> 5V_LNA1 (x2)
- C15 pad 1: 5V_LNA -> 5V_LNA1
- C16 pad 1: 5V_LNA -> 5V_LNA1
- C19 pad 1: 5V_LNA -> 5V_LNA1
- C20 pad 1: 5V_LNA -> 5V_LNA1
- C23 pad 1: GND -> 5V_LNA2
- C23 pad 2: Net-(U22-VOUT) -> GND
- C25 pad 1: 3.3V_IQ_DEMOD -> 5V_LNA2
- C37 pad 2: Net-(U5-CP) -> LO
- C46 pad 2: Net-(U12-BP) -> Net-(U17-BP)
- C48 pad 1: 5V_LNA -> 5V_LNA1
- C6 pad 1: Net-(C6-Pad1) -> Net-(U4-CLIN)
- C6 pad 2: Net-(C6-Pad2) -> GND
- C7 pad 2: GND -> Net-(U7-IF-)
- C8 pad 1: GND -> Net-(U4-RFOUT)
- C8 pad 2: Net-(U7-IF+) -> Net-(C8-Pad2)
- L10 pad 2: 5V_LNA -> 5V_LNA1
- L12 pad 1: Net-(C6-Pad2) -> Net-(U8-RFOUT)
- L12 pad 2: GND -> 5V_LNA2
- L8 pad 2: 5V_LNA -> 5V_LNA1 (x2)
- L9 pad 2: 5V_LNA -> 5V_LNA1
- R11 pad 1: DEMOD_I+ -> Net-(U12-TUNE)
- R11 pad 2: GND -> PWM_TUNE
- R30 pad 2: 5V_LNA -> 5V_LNA1
- R46 pad 2: 5V_ADC -> 3V3
- U12 pad 1: VIN -> Net-(U12-IND)
- U12 pad 3: VIN -> Net-(U12-TUNE)
- U12 pad 4: Net-(U12-BP) -> Net-(U12-OUT-)
- U12 pad 5: Net-(U12-VOUT) -> 3V3
- U15 pad 1: VIN -> Net-(U15-B)
- U15 pad 2: GND -> Net-(U16-C)
- U15 pad 3: VIN -> Net-(U15-C)
- U15 pad 4: Net-(U15-BP) -> Net-(U16-C)
- U21 pad 2: Net-(C6-Pad1) -> Net-(U4-RFIN)
- U23 pad 1: ADC_I_DB+ -> unconnected-(U23-Pad1)
- U23 pad 10: DEMOD_VCTRL -> unconnected-(U23-Pad10)
- U23 pad 2: ADC_I_DB- -> unconnected-(U23-Pad2)
- U23 pad 3: ADC_Q_CNV+ -> unconnected-(U23-Pad3)
- U23 pad 4: ADC_Q_CNV- -> unconnected-(U23-Pad4)
- U23 pad 7: ADC_Q_DCO+ -> unconnected-(U23-Pad7)
- U23 pad 8: ADC_Q_CLK- -> unconnected-(U23-Pad8)
- U23 pad 9: ADC_Q_CLK+ -> unconnected-(U23-Pad9)
- U4 pad 1: Net-(R16-Pad1) -> unconnected-(U4-NC-Pad1)
- U4 pad 2: Net-(C62-Pad2) -> Net-(U4-RFIN)
- U4 pad 3: LPF_I_VCM -> unconnected-(U4-NC-Pad3)
- U4 pad 4: -5V_OPAMP -> unconnected-(U4-NC-Pad4)
- U4 pad 5: -5V_OPAMP -> Net-(U4-CLIN)
- U4 pad 6: Net-(C63-Pad1) -> unconnected-(U4-NCIN-Pad6)
- U4 pad 7: 5V_OPAMP -> Net-(U4-RFOUT)
- U4 pad 8: 5V_OPAMP -> unconnected-(U4-NC-Pad8)
- U4 pad 9: unconnected-(U4-PAD-Pad9) -> GND
- U5 pad 1: GND -> VIN
- U5 pad 2: 3.3V_PMOD -> GND
- U5 pad 3: GND -> VIN
- U5 pad 4: 3.3V_PMOD -> Net-(U5-BP)
- U5 pad 5: 3.3V_PMOD -> Net-(U5-VOUT)
- U7 pad 1: GND -> Net-(C8-Pad2)
- U7 pad 2: Net-(U7-IF+) -> Net-(U8-RFIN)
- U9 pad 1: ADC_I_CNV+ -> ADC_SDI
- U9 pad 10: ADC_I_DCO+ -> PWM_TUNE
- U9 pad 2: ADC_I_CNV- -> unconnected-(U9-Pad2)
- U9 pad 3: ADC_I_CLK+ -> ADC_SCLK
- U9 pad 4: ADC_I_CLK- -> unconnected-(U9-Pad4)
- U9 pad 7: ADC_I_DA- -> ADC_SDO
- U9 pad 8: ADC_I_DA+ -> unconnected-(U9-Pad8)
- U9 pad 9: ADC_I_DCO- -> ADC_CONVST
Routing:
- net VIN: track 7.96 -> 110.2 mm
- net 5V_LNA1: track 0.00 -> 87.7 mm, vias 0 -> 27
- net 3V3: track 0.00 -> 64.5 mm, vias 0 -> 12
- net 5V_LNA2: track 0.00 -> 58.6 mm, vias 0 -> 22
- net GND: track 51.9 -> 86.9 mm, vias 87 -> 131
- net PWM_TUNE: track 0.00 -> 29.4 mm
- net 1V8: track 0.00 -> 26.7 mm, vias 0 -> 4
- net 5V_LNA: track 23.0 -> 0.00 mm, vias 10 -> 0
- net LO: track 0.00 -> 5.67 mm
- net Net-(U4-RFOUT): track 0.00 -> 5.23 mm
- net Net-(L13-Pad2): track 0.00 -> 5.09 mm
- net Net-(U8-RFOUT): track 0.00 -> 5.02 mm
- net Net-(U12-TUNE): track 0.00 -> 5.00 mm
- net Net-(U2-RFOUT): track 0.01 -> 4.89 mm
- net Net-(C4-Pad2): track 6.91 -> 2.16 mm
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Other:
- board text added: "TODO: Add copper zone here Layer 1 to Layer 4 connecting grounds"
- board text added: "TODO: Add solid GND planes on layers 2/3 Ground via stitching Decisions: Use 0.6x0.3 vias Use 0.3mm trace for 50ohm characteristic impedance for microstrip with solid groundplane in layers 2,3 oriented horizontally for EM fields Use 0.4mm silkscreen width/height to balance readability/placement Ensure RF Mixer (U4) is far away from sensitive RF/analog front end"
- board text removed: "TODO: Add solid GND planes on layers 2/3 Ground via stitching Decisions: Add ground stiching vias every lamba/10 to lambda/20 assuming er or 4.3 to 4.5 for FR4 which is 3.0 to 3.3mm for microstrip. Place vias every 3-5x trace width (1-1.2mm) Use 0.3mm trace for 50ohm characteristic impedance for microstrip with solid groundplane in layers 2,3 oriented horizontally for EM fields Use 0.4mm silkscre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"

Commit message: Final cleanup and GND planes for layers 2 and 3
Parts:
- removed the C10 at (38.0, 78.5)
- removed the C11 at (41.4, 82.5)
- removed the C12 at (35.3, 82.2)
- removed the C21 at (78.0, 100.1)
- removed the C22 at (137.6, 78.9)
- removed the C22 at (87.8, 80.0)
- removed the C24 at (82.8, 104.3)
- removed the C26 at (140.5, 75.0)
- removed the C26 at (90.3, 83.7)
- removed the C27 at (238.3, 97.3)
- removed the C28 at (90.2, 85.9)
- removed the C28 at (238.3, 99.2)
- removed the C29 at (87.6, 88.0)
- removed the C29 at (238.3, 101.2)
- removed the C30 at (140.5, 76.9)
- removed the C30 at (91.2, 95.3)
- removed the C30 at (220.0, 44.2)
- removed the C31 at (140.5, 78.9)
- removed the C31 at (91.2, 97.3)
- removed the C31 at (221.3, 44.5)
- removed the C32 at (93.1, 72.8)
- removed the C32 at (213.4, 43.7)
- removed the C33 at (143.9, 89.5)
- removed the C33 at (215.9, 43.2)
- removed the C34 at (228.9, 81.9)
- removed the C35 at (238.3, 107.1)
- removed the C36 at (68.5, 77.4)
- removed the C36 at (228.9, 84.9)
- removed the C38 at (71.8, 81.3)
- removed the C38 at (228.9, 87.9)
- removed the C39 at (238.3, 109.1)
- removed the C40 at (93.1, 76.7)
- removed the C40 at (228.9, 90.9)
- removed the C41 at (228.9, 93.9)
- removed the C41 at (90.7, 79.2)
- removed the C45 at (226.1, 76.1)
- removed the C47 at (228.9, 99.9)
- removed the C49 at (223.9, 88.8)
- removed the C49 at (118.5, 71.1)
- removed the C50 at (241.2, 99.2)
- removed the C51 at (223.9, 92.1)
- removed the C52 at (241.2, 101.2)
- removed C53, C94: 10u_50V, Capacitor_SMD:C_1206_3216Metric
- removed C54, C56, C57, C67, C69: 10u_16V, Capacitor_SMD:C_0805_2012Metric
- removed C55, C60 (x2), C72, C73, C74, C75, C81, C85, C88, C89, C90, C93: 0.1uF, Capacitor_SMD:C_0402_1005Metric
- removed C55, C56: 4.7u_16V, Capacitor_SMD:C_1206_3216Metric
- removed C57: 1u_16V, Capacitor_SMD:C_0603_1608Metric
- removed C58, C59, C80, C84: 100n_25V, Capacitor_SMD:C_0402_1005Metric
- removed C58, C59: 10n_25V, Capacitor_SMD:C_0402_1005Metric
- removed C61, C66, C78, C79: 10p_50V, Capacitor_SMD:C_0402_1005Metric
- removed C62, C65, C68, C76, C77, C82, C83: 1u_16V, Capacitor_SMD:C_0402_1005Metric
- removed C63, C64, C70, C71, C86, C87, C91, C92: 200p_50V, Capacitor_SMD:C_0402_1005Metric
- removed the C7 at (90.6, 75.2)
- removed D1: 1N5817, Diode_THT:D_DO-41_SOD81_P10.16mm_Horizontal
- removed D1, D3, D4 (x2): LED, LED_SMD:LED_0603_1608Metric
- removed the L13 at (144.4, 81.4)
- removed L14, L15: 72n, Inductor_SMD:L_0402_1005Metric
- removed L18: 10u, TheEEView_Footprint_Lib:SRU1028A-100Y
- removed the L6 at (232.6, 81.4)
- removed the L7 at (232.6, 83.4)
- removed the L8 at (41.9, 79.4)
- removed the R1 at (75.2, 78.0)
- removed the R11 at (232.8, 37.8)
- removed R12: 4.7kR, Resistor_SMD:R_0402_1005Metric
- removed R12, R2, R46: 150R, Resistor_SMD:R_0603_1608Metric
- removed R13, R14: 51R, Resistor_SMD:R_0402_1005Metric
- removed R13, R22, R40, R47: 49k3R, Resistor_SMD:R_0402_1005Metric
- removed R14, R23, R48, R49: 75kR, Resistor_SMD:R_0402_1005Metric
- removed R15, R25, R27, R28, R29, R38, R39: 50R, Resistor_SMD:R_0402_1005Metric
- removed R16: 51.1R, Resistor_SMD:R_0402_1005Metric
- removed R16, R24, R50, R52: 8k2R, Resistor_SMD:R_0402_1005Metric
- removed R17: 976R, Resistor_SMD:R_0402_1005Metric
- removed R17, R27, R54, R55: 2k43R, Resistor_SMD:R_0402_1005Metric
- removed R18, R25, R51, R53: 24R9, Resistor_SMD:R_0402_1005Metric
- removed R18, R19, R20: 1kR, Resistor_SMD:R_0402_1005Metric
- removed R19, R2, R28, R29: 20kR, Resistor_SMD:R_0402_1005Metric
- removed R20, R38, R39: 4k22R, Resistor_SMD:R_0402_1005Metric
- removed R21, R40: 50R, Resistor_SMD:R_0603_1608Metric
- removed R23, R24: 22R, Resistor_SMD:R_0603_1608Metric
- removed R26, R31, R32, R35: 0R, Resistor_SMD:R_0402_1005Metric
- removed R26, R32, R36, R37, R56, R57, R58, R59, R60, R61: 100R, Resistor_SMD:R_0402_1005Metric
- removed the R3 at (75.5, 81.9)
- removed R33: 130k, Resistor_SMD:R_0402_1005Metric
- removed R34: 300k, Resistor_SMD:R_0402_1005Metric
- removed R36: 100k, Resistor_SMD:R_0402_1005Metric
- removed R37: 66.5k, Resistor_SMD:R_0402_1005Metric
- removed the R4 at (75.5, 83.6)
- removed R41: 12kR, Resistor_SMD:R_0402_1005Metric
- removed R42: 5.6kR, Resistor_SMD:R_0402_1005Metric
- removed R43, R44: 470R, Resistor_SMD:R_0402_1005Metric
- removed the R5 at (75.5, 85.4)
- removed the R6 at (75.5, 87.7)
- removed the R7 at (76.6, 95.5)
- removed the R8 at (76.6, 97.5)
- removed the R9 at (76.6, 73.6)
- removed TP17: ~, TestPoint:TestPoint_Pad_D1.0mm
- removed the U10 at (237.2, 111.6)
- removed the U13 at (114.2, 89.8)
- removed the U13 at (254.8, 52.2)
- removed the U14 at (114.2, 96.7)
- removed the U16 at (216.8, 50.3)
- removed the U16 at (239.5, 39.8)
- removed the U17 at (112.7, 78.2)
- removed U22: ADL5531, TheEEView_Footprint_Lib:ADL5531
- removed U22: LP2985-3.3, Package_TO_SOT_SMD:SOT-23-5
- removed U23: PMOD 2x6, Connector_PinHeader_1.00mm:PinHeader_2x06_P1.00mm_Vertical
- removed U24: PAT1220-C-0DB, RF_Converter:RF_Attenuator_Susumu_PAT1220
- removed U24: ADA4899-1YRDZ, Package_SO:SOIC-8-1EP_3.9x4.9mm_P1.27mm_EP2.29x3mm_ThermalVias
- removed the U4 at (223.8, 38.5)
- removed the U6 at (242.0, 32.1)
- removed the U7 at (218.0, 43.7)
- removed the U8 at (238.4, 32.7)
- removed the U8 at (254.8, 45.6)
- added C22: 1n_50V, Capacitor_SMD:C_0402_1005Metric, F.Cu at (119.3, 42.7)
- moved TP22 121.6 mm to (102.4, 47.0)
- moved C6 41.6 mm to (109.2, 42.7), turned to 180 degrees
- moved U9 14.9 mm to (152.4, 30.2)
- moved C33 7.20 mm to (145.8, 36.5)
- moved R4 7.02 mm to (142.8, 33.9)
- moved C31 6.92 mm to (139.8, 31.7)
- moved C46 6.89 mm to (127.5, 31.7)
- moved C32 6.88 mm to (143.2, 32.2)
- moved C41 6.87 mm to (110.3, 31.2), turned to 180 degrees
- moved R7 6.79 mm to (130.3, 33.7)
- moved C49 6.75 mm to (133.3, 36.2)
- moved C47 6.70 mm to (130.8, 32.0)
- moved U17 6.70 mm to (128.9, 28.8)
- moved U5 6.70 mm to (141.3, 28.8)
- moved C30 6.46 mm to (140.7, 25.2)
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Routing:
- net 5V_LNA1: track 87.7 -> 41.7 mm, vias 27 -> 0
- net VIN: track 110.2 -> 145.4 mm
- net 5V_LNA2: track 58.6 -> 26.1 mm, vias 22 -> 0
- net PWM_TUNE: track 29.4 -> 46.3 mm
- net ADC_SDI: track 3.94 -> 18.9 mm
- net ADC_SCLK: track 3.79 -> 18.2 mm
- net 3V3: track 64.5 -> 50.4 mm, vias 12 -> 4
- net -2.5V_DiffAmp: track 12.3 -> 0.00 mm, vias 1 -> 0
- net ADC_SDO: track 4.42 -> 16.7 mm
- net ADC_CONVST: track 4.62 -> 16.2 mm
- net 1V8: track 26.7 -> 18.8 mm
- net Net-(U8--IN): track 7.24 -> 0.00 mm
- net Net-(U8-VOUT): track 6.46 -> 0.00 mm
- net GND: track 86.9 -> 80.9 mm, vias 131 -> 163
- net DIFF_OUTP: track 5.78 -> 0.00 mm
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- added copper zone on F.Cu, net GND
- added copper zone on In1.Cu, net GND
- added copper zone on In2.Cu, net GND
Other:
- board text added: "TODO: Add solid GND planes on layers 2/3 Ground via stitching Decisions: Use Coplanar Waveguide for RF filter section for more confined EM fields Use 0.6x0.3 vias Use 8mil trace with 0.05mm airgap assuming 1ounce copper, 4.6 dielectric constant Use 1mm via distance (2xgap) Use 2mm between vias horizontally for microstrip with solid groundplane in layers 2,3 oriented horizontally for EM fields Use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"
- board text removed: "TODO: Add solid GND planes on layers 2/3 Ground via stitching Decisions: Use 0.6x0.3 vias Use 0.3mm trace for 50ohm characteristic impedance for microstrip with solid groundplane in layers 2,3 oriented horizontally for EM fields Use 0.4mm silkscreen width/height to balance readability/placement Ensure RF Mixer (U4) is far away from sensitive RF/analog front end"

Commit message: Update textual comments and fix a via annular ring setting
Other:
- board text removed: "TODO: Add copper zone here Layer 1 to Layer 4 connecting grounds"
Changed lines of the file:
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@@
 		(layer "Margin")
 	)
-	(gr_text "TODO: Add copper zone \nhere Layer 1 to Layer 4 \nconnecting grounds"
-		(at 0.7 43.34 0)
-		(layer "Cmts.User")
-		(effects
-			(font
-				(size 0.8 0.8)
-				(thickness 0.1)
-			)
-			(justify left bottom)
-		)
-	)
 	(gr_text "12V lithium ion battery / or DC IN from benchtop power supply and GND"
 		(at 61.5 8.5 0)
@@
 		)
 	)
-	(gr_text "TODO: \nAdd solid GND planes on layers 2/3\nGround via stitching\nDecisions:\nUse Coplanar Waveguide for RF filter section for more confined EM fields \nUse 0.6x0.3 vias\nUse 8mil trace with 0.05mm airgap assuming 1ounce copper, 4.6 dielectric constant\nUse 1mm via distance (2xgap)\nUse 2mm between vias horizontally\nfor microstrip with solid groundplane in layers 2,3 oriented horizontally for EM fields\nUse 0.4mm silkscreen width/height to balance readability/placement\nEnsure RF Mixer (U4) is far away from sensitive RF/analog front end"
+	(gr_text "TODO: \nAdd solid GND planes on layers 2/3\nGround via stitching\nDecisions:\nUse Coplanar Waveguide for RF filter section for more confined EM fields \nUse 0.6x0.3 vias\nUse 8mil trace with 0.05mm airgap assuming 1ounce copper, 4.6 dielectric constant\nUse 1mm via distance (2xgap)\nUse 2mm between vias horizontally\nfor microstrip with solid groundplane in layers 2,3 oriented horizontally for EM fields\nUse 0.4mm silkscreen width/height to balance readability/placement\nEnsure RF Mixer (U12) is far away from sensitive RF/analog front end"
 		(at 49.7 6.6 0)
 		(layer "Cmts.User")
@@
 		(drill 0.3)
 		(layers "F.Cu" "B.Cu")
-		(remove_unused_layers yes)
-		(keep_end_layers yes)
 		(free yes)
-		(zone_layer_connections "In1.Cu" "In2.Cu")
 		(teardrops
 			(best_length_ratio 0.5)
@@
 	)
 	(zone
-		(net 2)
-		(net_name "GND")
-		(layer "F.Cu")
-		(name "$teardrop_padvia$")
-		(hatch none 0.1)
-		(priority 30138)
-		(attr
-			(teardrop
-				(type padvia)
-			)
-		)
-		(connect_pads yes
-			(clearance 0)
-		)
-		(min_thickness 0.0254)
-		(filled_areas_thickness no)
-		(fill yes
-			(thermal_gap 0.5)
-			(thermal_bridge_width 0.5)
-			(island_removal_mode 1)
-			(island_area_min 10)
-		)
-		(polygon
-			(pts
-				(xy 25.9909 40.434236) (xy 26.1941 40.434236) (xy 26.386736 39.898527) (xy 26.0925 39.839) (xy 25.798264 39.898527)
-			)
-		)
-	)
-	(zone
 		(net 76)
 		(net_name "Net-(U15-B)")
@@
 			)
 		)
+	)
+	(zone
+		(net 2)
+		(net_name "GND")
+		(layer "F.Cu")
+		(name "$teardrop_padvia$")
+		(hatch none 0.1)
+		(priority 30000)
+		(attr
+			(teardrop
+				(type padvia)
+			)
+		)
+		(connect_pads yes
+			(clearance 0)
+		)
+		(min_thickness 0.0254)
+		(filled_areas_thickness no)
+		(fill yes
+			(thermal_gap 0.5)
+			(thermal_bridge_width 0.5)
+			(island_removal_mode 1)
+			(island_area_min 10)
+		)
+		(polygon
+			(pts
+				(xy 25.9909 40.434236) (xy 26.1941 40.434236) (xy 26.386736 39.898527) (xy 26.0925 39.839) (xy 25.798264 39.898527)
+			)
+		)
