File: hardware/analog_front_end_v2.kicad_sch (KiCad schematic)
At the start: 105 parts, among them J1 Conn_Coaxial, J3 Conn_01x01_Socket, J4 Conn_01x01_Socket, U1 ADL5531, U10 MAX6002, U11 LP2985-5.0, U12 MAX2606, U13 PAT1220-C-0DB, U14 LP2985-5.0, U15 BFP540ESD, U16 BFP540ESD, U17 LP2985-3.3, U18 PAT1220-C-0DB, U19 PAT1220-C-0DB, U2 ADL5531, U20 PAT1220-C-0DB, U21 PAT1220-C-0DB, U22 MCP6286, U3 ADL5531, U4 ADL5531, U5 LP2985-1.8, U6 MCP33131, U7 PAT1220-C-0DB, U8 ADL5531, U9 PMOD 2x6 2.54mm pitch

Commit message: Move to KiCAD 10 and improve schematics readability
Other:
- moved on the sheet: C1, C2, C27, C28, C3, C4, C54, J1, L1, L2, L3, L4
